File: design-files/ASD2020.sch (EAGLE design)
At the start: 10 parts, among them J1 DF12-32-DP, J2 DF12-32-DS, SW1 PTS840 GKP, SW2 PTS840 GKP, U1 ATTINY88-MU

Commit message: update format
Parts:
- removed J3, J4: (no value), tinycircuits:AS-ITM-00235
- removed SW2: PTS840 GKP, tinycircuits:AS-ITM-00236
- added C3: 100uF, tinycircuits:AS-ITM-00095
- added C4: 10nF, tinycircuits:AS-ITM-00084
- added C6: 10uF, tinycircuits:AS-ITM-00002
- added J5, J6: FSM8JSMA, tinycircuits:AS-ITM-00278
- added J7: DM3D-SF, tinycircuits:AS-ITM-00047
- added Q1, Q2: DMP2035U, tinycircuits:AS-ITM-00024
- added R1: 1.00K, tinycircuits:AS-ITM-00008
- added R2, R4, R5, R6, R7: 100K, tinycircuits:AS-ITM-00004
- added SW5: 254SA104B50B, tinycircuits:AS-ITM-00229
- added U2: TS922IDT, tinycircuits:AS-ITM-000922
- added U3: W25Q64FVZPIG, tinycircuits:AS-ITM-00263
- C1: value 0.1uF -> 10uF; device tinycircuits:AS-ITM-00008 -> tinycircuits:AS-ITM-00002; PARTNO (none) -> AS-ITM-00002; VALUE (none) -> 10uF
- J1: value DF12-32-DP -> SKRHABE010; device tinycircuits:AS-ITM-00015 -> tinycircuits:AS-ITM-00305; PARTNO AS-ITM-00015 -> (none); VALUE DF12-32-DP -> (none)
- R3: value 10.0K -> 100K; device tinycircuits:AS-ITM-00032 -> tinycircuits:AS-ITM-00004; PARTNO (none) -> AS-ITM-00004; VALUE (none) -> 100K
- SW1: value PTS840 GKP -> PCM12SMTR; device tinycircuits:AS-ITM-00236 -> tinycircuits:AS-ITM-00220
- U1: value ATTINY88-MU -> SMT-0540-S-R; device tinycircuits:AS-ITM-00214 -> tinycircuits:AS-ITM-00144
Connections:
- removed net PC0: J4.X, U1.PC0(ADC0)
- removed net PC1: J4.Y, U1.PC1(ADC1)
- removed net PC2: J3.X, U1.PC2(ADC2)
- removed net PC3: J3.Y, U1.PC3(ADC3)
- removed net PD5: J3.VCC, U1.PD5
- removed net PD6: J4.VCC, U1.PC7
- removed net SW0: SW1.2, U1.PD2(INT0)
- removed net SW1: SW2.2, U1.PD3(INT1)
- new net AUDIOIN: SW1.2, U2.IN1+
- new net N$1: C3.1, U2.2IN-, U2.2OUT
- new net N$12: J1.B, Q1.G, R3.1
- new net N$13: J1.D, Q2.G, R2.1
- new net N$2: C3.2, U1.+LEAD
- new net N$4: SW5.S2
- new net N$7: C4.1, R1.2, U2.2IN+
- new net N$9: R1.1, U2.IN1-, U2.OUT1
- new net SW3: SW5.S1
- net +3V3: no longer J1.6
- net +5V: no longer J1.8
- net AD0: now also SW1.1; no longer J1.11
- net AD1: now also J1.C, Q1.D, R4.1, R5.2, SW5.A2; no longer J1.9
- net AD2: no longer J1.7
- net AD3: no longer J1.5
- net AD4/SDA: no longer J1.3, U1.PC4(SDA)
- net AD5/SCL: no longer J1.1, U1.PC5(SCL)
- net AREF: now also J1.A, Q2.D, R6.1, R7.2, SW5.B2; no longer J1.13
- net GND: now also C4.2, C6.2, J1.CMN, J5.2, J6.2, J7.VSS, R5.1, R7.1, SW1.3, SW5.A1, SW5.B3, U1.-LEAD, U2.VCC-, U3.GND; no longer J1.12, J1.14, J3.GND, J4.GND, SW1.1, SW2.1, U1.GND, U1.GND1, U1.PAD
- net IO0: no longer J1.24
- net IO1: no longer J1.26
- net IO2: no longer J1.28
- net IO3: no longer J1.30
- net IO4: no longer J1.32
- net IO5: now also U3./CS; no longer J1.31
- net IO6: no longer J1.29
- net IO7: no longer J1.27
- net IO8: no longer J1.25
- net IO9: no longer J1.23
- net MISO: now also J7.DAT0, U3.DO; no longer J1.17, U1.PB4(MISO)
- net MOSI: now also J7.CMD, U3.DI; no longer J1.19, U1.PB3(MOSI)
- net RESET: no longer J1.22, R3.2, U1.PC6(RESET)
- net RSV0: now also J5.3; no longer J1.20
- net RSV1: now also J6.3; no longer J1.18
- net RSV2: no longer J1.16
- net SCK: now also J7.CLK, U3.CLK; no longer J1.15, U1.PB5(SCK)
- net SS: now also J7.CD/DAT3; no longer J1.21
- net VBATT: no longer J1.4
- net VCC: now also C6.1, J7.VDD, Q1.S, Q2.S, R2.2, R3.2, R4.2, R6.2, SW5.A3, SW5.B1, U2.VCC+, U3./HOLD, U3./WP, U3.VCC; no longer J1.2, R3.1, U1.AVCC, U1.VCC
- net VIN: no longer J1.10
Other:
- note added: "17,17.5 63,17.5"
- note added: "4"
- note added: "Down"
- note added: "Left"
- note added: "Right"
- note added: "pick better buttons?"
- note added: "smt?"
- note added: "speaker- JST or?"
- note added: "up"
- note added: "x"
- note added: "y"
- note removed: "3"
- note removed: "TinyShield Expansion - Top"
- moved on the sheet: C1, C2, R3
